Commit message: It mostly works

File: src/sam_bot_nav2_gz/description/rover_2wd.urdf (robot description, URDF)
Before this commit: robot rover_2wd, 7 links, 6 joints
Links:
- removed link front_caster
- added link chassis_link, mass ${chassis_mass}; collision mesh filename=file://$(find sam_bot_nav2_gz)/models/rover/rover_2wd_core.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; visual mesh filename=file://$(find sam_bot_nav2_gz)/models/rover/rover_2wd_core.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
- added link fl_wheel_link, mass ${wheel_mass}; collision mesh filename=file://$(find sam_bot_nav2_gz)/models/rover/pro_tire.dae; visual mesh filename=file://$(find sam_bot_nav2_gz)/models/rover/pro_tire.dae
- added link fr_wheel_link, mass ${wheel_mass}; collision mesh filename=file://$(find sam_bot_nav2_gz)/models/rover/pro_tire.dae; visual mesh filename=file://$(find sam_bot_nav2_gz)/models/rover/pro_tire.dae
- added link rl_castor_housing_link, mass ${castor_housing_mass}; collision mesh filename=file://$(find sam_bot_nav2_gz)/models/rover/castor_housing.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; visual mesh filename=file://$(find sam_bot_nav2_gz)/models/rover/castor_housing.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
- added link rl_castor_link, mass ${castor_mass}; collision mesh filename=file://$(find sam_bot_nav2_gz)/models/rover/castor.dae; visual mesh filename=file://$(find sam_bot_nav2_gz)/models/rover/castor.dae
- added link rr_castor_housing_link, mass ${castor_housing_mass}; collision mesh filename=file://$(find sam_bot_nav2_gz)/models/rover/castor_housing.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; visual mesh filename=file://$(find sam_bot_nav2_gz)/models/rover/castor_housing.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
- added link rr_castor_link, mass ${castor_mass}; collision mesh filename=file://$(find sam_bot_nav2_gz)/models/rover/castor.dae; visual mesh filename=file://$(find sam_bot_nav2_gz)/models/rover/castor.dae
- link base_link: geometry 
Joints:
- removed joint caster_joint
- added joint base_to_chassis: type fixed, parent base_link, child chassis_link, origin xyz=0 0 0.125
- added joint fl_wheel_to_chassis: type continuous, parent chassis_link, child fl_wheel_link, origin xyz=${wheel_x_offset} ${wheel_y_offset} 0 rpy=0 0 0, axis 0 1 0
- added joint fr_wheel_to_chassis: type continuous, parent chassis_link, child fr_wheel_link, origin xyz=${wheel_x_offset} ${-wheel_y_offset} 0 rpy=0 0 0, axis 0 1 0
- added joint rl_castor_to_chassis: type continuous, parent rl_castor_housing_link, child rl_castor_link, origin xyz=-0.031 0 -0.027 rpy=0 0 0, axis 0 1 0
- added joint rl_ch_to_chassis: type continuous, parent chassis_link, child rl_castor_housing_link, origin xyz=${-wheel_x_offset - castor_x_offset} ${castor_y_offset + 0.0025} ${castor_z_offset} rpy=0 0 0, axis 0 0 1
- added joint rr_castor_to_chassis: type continuous, parent rr_castor_housing_link, child rr_castor_link, origin xyz=-0.031 0 -0.027 rpy=0 0 0, axis 0 1 0
- added joint rr_ch_to_chassis: type continuous, parent chassis_link, child rr_castor_housing_link, origin xyz=${-wheel_x_offset - castor_x_offset} ${-castor_y_offset} ${castor_z_offset} rpy=0 0 0, axis 0 0 1

File: src/sam_bot_nav2_gz/description/rover_dev_payload.urdf (robot description, URDF)
Before this commit: robot rover_miti_payload, 1 links, 1 joints
Links:
- link payload_link: geometry collision mesh filename=file://$(find sam_bot_nav2_gz)/models/rover/rover_payload.d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; visual mesh filename=file://$(find sam_bot_nav2_gz)/models/rover/rover_payload.d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

Commit message: Nav works, gz doesn't

File: src/sam_bot_nav2_gz/description/rover_2wd.urdf (robot description, URDF)
Before this commit: robot rover_2wd, 13 links, 12 joints
Joints:
- joint base_joint: origin xyz=0.0 0.0 ${-(wheel_radius+wheel_zoff)} rpy=0 0 0 -> xyz=0.0 0.0 -0.15 rpy=0 0 0
- joint lidar_joint: origin xyz=0 0 0.12 rpy=0 0 0 -> xyz=0 0 0.3 rpy=0 0 0

Commit message: Fix IMU placement

File: src/sam_bot_nav2_gz/description/rover_2wd.urdf (robot description, URDF)
Before this commit: robot rover_2wd, 13 links, 12 joints
Joints:
- joint imu_joint: origin xyz=0 0 0.01 -> xyz=0 0 0.1

Commit message: Use the Rover IMU. Remove camera.

File: src/sam_bot_nav2_gz/description/rover_2wd.urdf (robot description, URDF)
Before this commit: robot rover_2wd, 13 links, 12 joints
Links:
- removed link camera_frame
- removed link camera_link
- removed link imu_link
Joints:
- removed joint camera_frame_joint
- removed joint camera_joint
- removed joint imu_joint
- joint lidar_joint: origin xyz=0 0 0.3 rpy=0 0 0 -> xyz=0 0 0.5 rpy=0 0 0
