Commit message: Directory restructuring. Rename sam_bot_nav2 -> nav2_gazebo

File: description/lidar.urdf (robot description, URDF)
Before this commit: robot rplidar_s2, 1 links, 1 joints
Links:
- link lidar_link: geometry collision mesh filename=file://$(find nav2_gazebo)/models/rover/rplidar_s2.dae; visual mesh filename=file://$(find nav2_gazebo)/models/rover/rplidar_s2.dae

File: description/rover_2wd.urdf (robot description, URDF)
Before this commit: robot rover_2wd, 10 links, 9 joints
Links:
- link chassis_link: geometry collision mesh filename=file://$(find nav2_gazebo)/models/rover/rover_2wd_core.dae; visual mesh filename=file://$(find nav2_gazebo)/models/rover/rover_2wd_core.dae
- link fl_wheel_link: geometry collision mesh filename=file://$(find nav2_gazebo)/models/rover/pro_tire.dae; visual mesh filename=file://$(find nav2_gazebo)/models/rover/pro_tire.dae
- link fr_wheel_link: geometry collision mesh filename=file://$(find nav2_gazebo)/models/rover/pro_tire.dae; visual mesh filename=file://$(find nav2_gazebo)/models/rover/pro_tire.dae
- link rl_castor_housing_link: geometry collision mesh filename=file://$(find nav2_gazebo)/models/rover/castor_housing.dae; visual mesh filename=file://$(find nav2_gazebo)/models/rover/castor_housing.dae
- link rl_castor_link: geometry collision mesh filename=file://$(find nav2_gazebo)/models/rover/castor.dae; visual mesh filename=file://$(find nav2_gazebo)/models/rover/castor.dae
- link rr_castor_housing_link: geometry collision mesh filename=file://$(find nav2_gazebo)/models/rover/castor_housing.dae; visual mesh filename=file://$(find nav2_gazebo)/models/rover/castor_housing.dae
- link rr_castor_link: geometry collision mesh filename=file://$(find nav2_gazebo)/models/rover/castor.dae; visual mesh filename=file://$(find nav2_gazebo)/models/rover/castor.dae

File: description/rover_dev_payload.urdf (robot description, URDF)
Before this commit: robot rover_miti_payload, 1 links, 1 joints
Links:
- link payload_link: geometry collision mesh filename=file://$(find nav2_gazebo)/models/rover/rover_payload.dae; visual mesh filename=file://$(find nav2_gazebo)/models/rover/rover_payload.dae
