Commit message: Add latching lever

File: description/rover_2wd.urdf (robot description, URDF)
Before this commit: robot rover_2wd, 10 links, 9 joints
Links:
- added link latch_lever; collision cylinder length=0.6 radius=0.02; visual cylinder length=0.6 radius=0.02
Joints:
- added joint base_to_latch_lever: type fixed, parent base_link, child latch_lever, origin xyz=0.5 0 0.3 rpy=0 1.57123 0
- joint lidar_joint: origin xyz=0 0 0.5 rpy=0 0 0 -> xyz=0 0 0.4 rpy=0 0 0

Commit message: Add contact and touch sensor

File: description/rover_2wd.urdf (robot description, URDF)
Before this commit: robot rover_2wd, 11 links, 10 joints
Joints:
- joint base_to_latch_lever: parent base_link -> chassis_link

Commit message: Updates

File: description/rover_2wd.urdf (robot description, URDF)
Before this commit: robot rover_2wd, 11 links, 10 joints
Links:
- link latch_lever: geometry collision cylinder length=0.6 radius=0.02
Joints:
- joint base_to_latch_lever: origin xyz=0.5 0 0.3 rpy=0 1.57123 0 -> xyz=-0.5 0 0.15 rpy=0 1.57123 0

Commit message: Update latch lever pose

File: description/rover_2wd.urdf (robot description, URDF)
Before this commit: robot rover_2wd, 11 links, 10 joints
Links:
- link latch_lever: geometry collision cylinder length=0.6 radius=0.02; visual cylinder length=0.6 radius=0.02
Joints:
- joint base_to_latch_lever: origin xyz=-0.5 0 0.15 rpy=0 1.57123 0 -> xyz=-0.5 0 0.5 rpy=1.57123 0 0

Commit message: Config updates

File: description/rover_2wd.urdf (robot description, URDF)
Before this commit: robot rover_2wd, 11 links, 10 joints
Links:
- link latch_lever: geometry collision cylinder length=0.6 radius=0.02

Commit message: Tune navigation and add latch visual

File: description/rover_2wd.urdf (robot description, URDF)
Before this commit: robot rover_2wd, 11 links, 10 joints
Links:
- added link latch_lever_visual_left; visual cylinder length=0.6 radius=0.02
- added link latch_lever_visual_right; visual cylinder length=0.6 radius=0.02
- link latch_lever: geometry collision cylinder length=0.4 radius=0.02
Joints:
- added joint base_to_latch_visual_left: type fixed, parent chassis_link, child latch_lever_visual_left, origin xyz=-0.5 -0.16 0.18 rpy=0 1.57123 0
- added joint base_to_latch_visual_right: type fixed, parent chassis_link, child latch_lever_visual_right, origin xyz=-0.5 0.16 0.18 rpy=0 1.57123 0
- joint base_to_latch_lever: origin xyz=-0.5 0 0.5 rpy=1.57123 0 0 -> xyz=-0.5 0 0.5 rpy= 0 1.57123 0
